File: 2015/comp_details/coin_sensor_board/coinsensor_pcb/capsense_coin.sch (EAGLE design)
At the start: 41 parts, among them J1 CON_HEADER_1X08, Q1 MOSFET-NCHANNELBSS123LT1G, Q2 MOSFET-NCHANNELBSS123LT1G, U1 CY8C4125AXI-483

Commit message: Update capsense with values
Parts:
- C5: value (none) -> 100n
- C8: value 10nF -> DNM
- Q1, Q2: value MOSFET-NCHANNELBSS123LT1G -> IRLML2502PFCNT-ND
- R1, R13, R14, R16, R17: value (none) -> DNM
- R10, R11, R12: value 100R -> 51R
- R15: value (none) -> 10k
- R2, R3, R4, R5, R6, R7, R8, R9: value (none) -> 200R
Other:
- note added: "Programming requires: SWDIO, SWDCLK, XRES, VCC, GND"
- note added: "R13/R14 mounted for I2C operation R16/R17 mounted for 'terminating' coin only on I2C bus"
- note added: "Shield Tank Cap (10nF, Optional)"
- note added: "TODO: Check value of C2, might need to reduce it for our uses?"
- note removed: "Shield Tank Cap (Optional)"
- moved on the sheet: R10, R11, R12, R13, R16, R17
