File: 2015/comp_details/course_layout.brd (EAGLE design)
At the start: 0 parts

Commit message: Updates
Routing:
- net S$1: track 219.5 -> 239.3 mm
- net S$7: track 0.00 -> 15.2 mm
- net S$4: track 0.00 -> 15.2 mm
- net S$6: track 0.00 -> 12.2 mm
- net S$5: track 0.00 -> 12.2 mm
Changed lines of the file:
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@@
 <?xml version="1.0" encoding="utf-8"?>
 <!DOCTYPE eagle SYSTEM "eagle.dtd">
-<eagle version="7.2.0">
+<eagle version="7.3.0">
 <drawing>
 <settings>
@@
 <setting verticaltext="up"/>
 </settings>
-<grid distance="0.06" unitdist="inch" unit="inch" style="lines" multiple="1" display="no" altdistance="0.025" altunitdist="inch" altunit="inch"/>
+<grid distance="0.03" unitdist="inch" unit="inch" style="lines" multiple="1" display="no" altdistance="0.025" altunitdist="inch" altunit="inch"/>
 <layers>
 <layer number="1" name="Top" color="4" fill="1" visible="yes" active="yes"/>
@@
 <rectangle x1="14.859" y1="0" x2="19.05" y2="1.143" layer="21" rot="R180"/>
 <circle x="16.764" y="1.143" radius="0.381" width="0.508" layer="104"/>
+<wire x1="32.004" y1="59.436" x2="32.004" y2="54.864" width="0.762" layer="101"/>
+<wire x1="13.716" y1="59.436" x2="13.716" y2="54.864" width="0.762" layer="101"/>
+<wire x1="11.684" y1="48.26" x2="13.716" y2="48.26" width="0.762" layer="101"/>
+<wire x1="24.384" y1="33.528" x2="24.384" y2="36.068" width="0.762" layer="101"/>
+<wire x1="27.432" y1="30.48" x2="30.48" y2="30.48" width="0.762" layer="101"/>
+<wire x1="21.336" y1="30.48" x2="18.288" y2="30.48" width="0.762" layer="101"/>
+<wire x1="24.384" y1="27.432" x2="24.384" y2="24.892" width="0.762" layer="101"/>
+<wire x1="26.416" y1="28.448" x2="28.448" y2="26.416" width="0.762" layer="101"/>
+<wire x1="26.416" y1="32.512" x2="28.448" y2="34.544" width="0.762" layer="101"/>
+<wire x1="22.352" y1="32.512" x2="20.32" y2="34.544" width="0.762" layer="101"/>
+<wire x1="22.352" y1="28.448" x2="20.32" y2="26.416" width="0.762" layer="101"/>
+<wire x1="37.592" y1="12.7" x2="35.56" y2="12.7" width="0.762" layer="101"/>
+<wire x1="35.052" y1="1.524" x2="35.052" y2="6.096" width="0.762" layer="101"/>
+<wire x1="16.764" y1="1.524" x2="16.764" y2="6.096" width="0.762" layer="101"/>
 </plain>
 <attributes>
@@
 <signals>
 <signal name="S$1">
-<wire x1="0" y1="0" x2="0" y2="60.96" width="0.508" layer="1"/>
+<wire x1="0" y1="0" x2="0" y2="22.098" width="0.508" layer="1"/>
+<wire x1="0" y1="22.098" x2="0" y2="24.384" width="0.508" layer="1"/>
+<wire x1="0" y1="24.384" x2="0" y2="60.96" width="0.508" layer="1"/>
 <wire x1="0" y1="60.96" x2="48.768" y2="60.96" width="0.508" layer="1"/>
-<wire x1="48.768" y1="60.96" x2="48.768" y2="0" width="0.508" layer="1"/>
+<wire x1="48.768" y1="60.96" x2="48.768" y2="38.862" width="0.508" layer="1"/>
+<wire x1="48.768" y1="38.862" x2="48.768" y2="36.576" width="0.508" layer="1"/>
+<wire x1="48.768" y1="36.576" x2="48.768" y2="0" width="0.508" layer="1"/>
 <wire x1="48.768" y1="0" x2="0" y2="0" width="0.508" layer="1"/>
+<wire x1="44.958" y1="38.862" x2="48.768" y2="38.862" width="0.762" layer="1"/>
+<wire x1="44.958" y1="38.862" x2="44.958" y2="36.576" width="0.762" layer="1"/>
+<wire x1="44.958" y1="36.576" x2="48.768" y2="36.576" width="0.762" layer="1"/>
+<wire x1="0" y1="22.098" x2="3.81" y2="22.098" width="0.762" layer="1"/>
+<wire x1="3.81" y1="22.098" x2="3.81" y2="24.384" width="0.762" layer="1"/>
+<wire x1="3.81" y1="24.384" x2="0" y2="24.384" width="0.762" layer="1"/>
 </signal>
 <signal name="S$2">
@@
 <via x="15.748" y="19.812" extent="1-16" drill="0.001" diameter="1"/>
 </signal>
+<signal name="S$4">
+<wire x1="28.194" y1="47.244" x2="32.004" y2="47.244" width="0.762" layer="1"/>
+<wire x1="32.004" y1="47.244" x2="32.004" y2="43.434" width="0.762" layer="1"/>
+<wire x1="32.004" y1="43.434" x2="28.194" y2="43.434" width="0.762" layer="1"/>
+<wire x1="28.194" y1="43.434" x2="28.194" y2="47.244" width="0.762" layer="1"/>
+</signal>
+<signal name="S$5">
+<wire x1="28.194" y1="38.862" x2="32.004" y2="38.862" width="0.762" layer="1"/>
+<wire x1="32.004" y1="38.862" x2="32.004" y2="36.576" width="0.762" layer="1"/>
+<wire x1="32.004" y1="36.576" x2="28.194" y2="36.576" width="0.762" layer="1"/>
+<wire x1="28.194" y1="36.576" x2="28.194" y2="38.862" width="0.762" layer="1"/>
+</signal>
+<signal name="S$6">
+<wire x1="16.764" y1="24.384" x2="20.574" y2="24.384" width="0.762" layer="1"/>
+<wire x1="20.574" y1="24.384" x2="20.574" y2="22.098" width="0.762" layer="1"/>
+<wire x1="20.574" y1="22.098" x2="16.764" y2="22.098" width="0.762" layer="1"/>
+<wire x1="16.764" y1="22.098" x2="16.764" y2="24.384" width="0.762" layer="1"/>
+</signal>
+<signal name="S$7">
+<wire x1="16.764" y1="17.526" x2="20.574" y2="17.526" width="0.762" layer="1"/>
+<wire x1="20.574" y1="17.526" x2="20.574" y2="13.716" width="0.762" layer="1"/>
+<wire x1="20.574" y1="13.716" x2="16.764" y2="13.716" width="0.762" layer="1"/>
+<wire x1="16.764" y1="13.716" x2="16.764" y2="17.526" width="0.762" layer="1"/>
+</signal>
 </signals>
